File: PCB/ESPLEDDriver.kicad_pcb (KiCad board)
At the start: 2 copper layers, 58.3 x 54.8 mm, 37 parts, among them J1 Conn_01x04_Pin, J2 Screw_Terminal_01x02, J3 Screw_Terminal_01x05, J4 Screw_Terminal_01x03, J5 Conn_01x20_Socket, Q1 IRLR2705, Q2 IRLR2705, Q3 IRLR2705, Q4 IRLR2705, U1 ESP32-C3-WROOM-02, U2 XL1509-3.3

Commit message: created case, finalized pcb (for realsies this time)
Parts:
- added G***: LOGO, LOGO, F.Cu at (71.5, 90.1)
- added G***: LOGO, LOGO, B.Cu at (70.7, 87.9)
- moved G*** 0.22 mm to (65.3, 88.0)

Commit message: slightly modified schematic and pcb due to incorrect screw terminal footprint
Parts:
- J2: footprint TerminalBlock_Phoenix:TerminalBlock_Phoenix_MKDS-1,5-2_1x02_P5.00mm_Horizontal -> TerminalBlock_Phoenix:TerminalBlock_Phoenix_PT-1,5-2-5.0-H_1x02_P5.00mm_Horizontal
- J3: footprint TerminalBlock_Phoenix:TerminalBlock_Phoenix_MKDS-1,5-5_1x05_P5.00mm_Horizontal -> TerminalBlock_Phoenix:TerminalBlock_Phoenix_PT-1,5-5-5.0-H_1x05_P5.00mm_Horizontal
- J4: footprint TerminalBlock_Phoenix:TerminalBlock_Phoenix_MKDS-1,5-3_1x03_P5.00mm_Horizontal -> TerminalBlock_Phoenix:TerminalBlock_Phoenix_PT-1,5-3-5.0-H_1x03_P5.00mm_Horizontal
